File: PCB/Rocket_solder.kicad_pcb (KiCad board)
At the start: 2 copper layers, 73.7 x 89.2 mm, 38 parts, among them M1 Motor_DC, Q1 2N3904, Q2 2N3904, Q3 2N3904, Q4 2N3904, Q5 2N3904, Q6 2N3904, Q7 2N3904, Q8 2N3904, SW1 SW_Push, U1 LM555xN

Commit message: updated pcb
Parts:
- added ?: LOGO, Rocket_solder:moon,, B.Cu at (200.0, 52.0)
- added ?: LOGO, Rocket_solder5:hmm, B.Cu at (196.0, 62.0)
- added G***: LOGO, Rocket_solder3:qr_insta, F.Cu at (205.0, 59.0)
- added G***: LOGO, Rocket_solder2:purrrr, B.Cu at (206.4, 57.7)
- D2: value LED -> POWER
- moved Q3 8.98 mm to (219.5, 66.0)
- moved D2 4.49 mm to (208.7, 53.0)
- renumbered G*** to ?
Routing:
- net /CLK_OUT: track 118.1 -> 111.3 mm, vias 0 -> 1
- net Net-(Q3-C): track 19.4 -> 14.3 mm
- net +6V: track 170.2 -> 174.3 mm
- net /LIGHT_ENABLE: track 108.4 -> 104.5 mm, vias 1 -> 0
- net Net-(BT1-+): track 28.1 -> 25.1 mm
