File: PCB/Rocket_solder.kicad_sch (KiCad schematic)
At the start: 33 parts, among them M1 Motor_DC, Q1 2N3904, Q2 2N3904, Q3 2N3904, Q4 2N3904, Q5 2N3904, Q6 2N3904, Q7 2N3904, Q8 2N3904, SW1 SW_Push, U1 LM555xN

Commit message: updated pcb
Parts:
- BT1, BT2: value Battery_Cell -> 3
- Q1, Q2, Q3, Q4, Q5, Q6, Q7, Q8: value 2N3904 -> 10u
Changed lines of the file:
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@@
 			)
 		)
-		(property "Value" "2N3904"
+		(property "Value" "10u"
 			(at 133.35 124.4599 0)
 			(show_name no)
@@
 			)
 		)
-		(property "Value" "2N3904"
+		(property "Value" "10u"
 			(at 182.88 69.8499 0)
 			(show_name no)
@@
 			)
 		)
-		(property "Sim.Pins" "1=E 2=B 3=C"
+		(property "Sim.Pins" "1=C 2=B 3=E"
+			(at 177.8 68.58 0)
+			(hide yes)
+			(show_name no)
+			(do_not_autoplace no)
+			(effects
+				(font
+					(size 1.27 1.27)
+				)
+			)
+		)
+		(property "Sim.Type" "GUMMELPOON"
 			(at 177.8 68.58 0)
 			(hide yes)
@@
 			)
 		)
-		(property "Value" "2N3904"
+		(property "Value" "10u"
 			(at 158.75 72.3899 0)
 			(show_name no)
@@
 			)
 		)
-		(property "Sim.Pins" "1=E 2=B 3=C"
+		(property "Sim.Pins" "1=C 2=B 3=E"
+			(at 153.67 71.12 0)
+			(hide yes)
+			(show_name no)
+			(do_not_autoplace no)
+			(effects
+				(font
+					(size 1.27 1.27)
+				)
+			)
+		)
+		(property "Sim.Type" "GUMMELPOON"
 			(at 153.67 71.12 0)
 			(hide yes)
@@
 			)
 		)
-		(property "Sim.Pins" "1=K 2=A"
+		(property "Sim.Pins" "1=A 2=K"
+			(at 171.45 48.26 0)
+			(hide yes)
+			(show_name no)
+			(do_not_autoplace no)
+			(effects
+				(font
+					(size 1.27 1.27)
+				)
+			)
+		)
+		(property "Sim.Device" "D"
 			(at 171.45 48.26 0)
 			(hide yes)
@@
 			)
 		)
-		(property "Value" "2N3904"
+		(property "Value" "10u"
 			(at 144.78 72.3899 0)
 			(show_name no)
@@
 			)
 		)
-		(property "Sim.Pins" "1=E 2=B 3=C"
+		(property "Sim.Pins" "1=C 2=B 3=E"
+			(at 139.7 71.12 0)
+			(hide yes)
+			(show_name no)
+			(do_not_autoplace no)
+			(effects
+				(font
+					(size 1.27 1.27)
+				)
+			)
+		)
+		(property "Sim.Type" "GUMMELPOON"
 			(at 139.7 71.12 0)
 			(hide yes)
@@
 			)
 		)
-		(property "Sim.Pins" "1=K 2=A"
+		(property "Sim.Pins" "1=A 2=K"
+			(at 127 48.26 0)
+			(hide yes)
+			(show_name no)
+			(do_not_autoplace no)
+			(effects
+				(font
+					(size 1.27 1.27)
+				)
+			)
+		)
+		(property "Sim.Device" "D"
 			(at 127 48.26 0)
 			(hide yes)
@@
 			)
 		)
-		(property "Value" "2N3904"
+		(property "Value" "10u"
 			(at 168.91 69.8499 0)
 			(show_name no)
@@
 			)
 		)
-		(property "Sim.Pins" "1=E 2=B 3=C"
+		(property "Sim.Pins" "1=C 2=B 3=E"
+			(at 163.83 68.58 0)
+			(hide yes)
+			(show_name no)
+			(do_not_autoplace no)
+			(effects
+				(font
+					(size 1.27 1.27)
+				)
+			)
+		)
+		(property "Sim.Type" "GUMMELPOON"
 			(at 163.83 68.58 0)
 			(hide yes)
@@
 			)
 		)
-		(property "Sim.Pins" "1=K 2=A"
+		(property "Sim.Pins" "1=A 2=K"
+			(at 161.29 48.26 0)
+			(hide yes)
+			(show_name no)
+			(do_not_autoplace no)
+			(effects
+				(font
+					(size 1.27 1.27)
+				)
+			)
+		)
+		(property "Sim.Device" "D"
 			(at 161.29 48.26 0)
 			(hide yes)
@@
 			)
 		)
-		(property "Value" "Battery_Cell"
+		(property "Value" "3"
 			(at 81.28 94.6784 0)
 			(show_name no)
@@
 			)
 		)
-		(property "Sim.Pins" "1=K 2=A"
+		(property "Sim.Pins" "1=A 2=K"
+			(at 149.86 48.26 0)
+			(hide yes)
+			(show_name no)
+			(do_not_autoplace no)
+			(effects
+				(font
+					(size 1.27 1.27)
+				)
+			)
+		)
+		(property "Sim.Device" "D"
 			(at 149.86 48.26 0)
 			(hide yes)
@@
 			)
 		)
-		(property "Value" "2N3904"
+		(property "Value" "10u"
 			(at 196.85 69.8499 0)
 			(show_name no)
@@
 			)
 		)
-		(property "Sim.Pins" "1=E 2=B 3=C"
+		(property "Sim.Pins" "1=C 2=B 3=E"
+			(at 191.77 68.58 0)
+			(hide yes)
+			(show_name no)
+			(do_not_autoplace no)
+			(effects
+				(font
+					(size 1.27 1.27)
+				)
+			)
+		)
+		(property "Sim.Type" "GUMMELPOON"
 			(at 191.77 68.58 0)
 			(hide yes)
@@
 			)
 		)
-		(property "Sim.Pins" "1=K 2=A"
+		(property "Sim.Pins" "1=A 2=K"
+			(at 138.43 48.26 0)
+			(hide yes)
+			(show_name no)
+			(do_not_autoplace no)
+			(effects
+				(font
+					(size 1.27 1.27)
+				)
+			)
+		)
+		(property "Sim.Device" "D"
 			(at 138.43 48.26 0)
 			(hide yes)
@@
 			)
 		)
-		(property "Value" "2N3904"
+		(property "Value" "10u"
 			(at 130.81 73.6599 0)
 			(show_name no)
@@
 			)
 		)
-		(property "Sim.Pins" "1=E 2=B 3=C"
+		(property "Sim.Pins" "1=C 2=B 3=E"
+			(at 125.73 72.39 0)
+			(hide yes)
+			(show_name no)
+			(do_not_autoplace no)
+			(effects
+				(font
+					(size 1.27 1.27)
+				)
+			)
+		)
+		(property "Sim.Type" "GUMMELPOON"
 			(at 125.73 72.39 0)
 			(hide yes)
@@
 			)
 		)
-		(property "Value" "Battery_Cell"
+		(property "Value" "3"
 			(at 60.96 94.6784 0)
 			(show_name no)
@@
 			)
 		)
-		(property "Sim.Pins" "1=K 2=A"
+		(property "Sim.Pins" "1=A 2=K"
+			(at 182.88 48.26 0)
+			(hide yes)
+			(show_name no)
+			(do_not_autoplace no)
+			(effects
+				(font
+					(size 1.27 1.27)
+				)
+			)
+		)
+		(property "Sim.Device" "D"
 			(at 182.88 48.26 0)
 			(hide yes)
@@
 			)
 		)
-		(property "Value" "2N3904"
+		(property "Value" "10u"
 			(at 73.66 76.1999 0)
 			(show_name no)
@@
 			)
 		)
-		(property "Sim.Pins" "1=E 2=B 3=C"
+		(property "Sim.Pins" "1=C 2=B 3=E"
+			(at 68.58 74.93 0)
+			(hide yes)
+			(show_name no)
+			(do_not_autoplace no)
+			(effects
+				(font
+					(size 1.27 1.27)
+				)
+			)
+		)
+		(property "Sim.Type" "GUMMELPOON"
 			(at 68.58 74.93 0)
 			(hide yes)
